File: Control PCB/control/control.kicad_sch (KiCad schematic)
At the start: 123 parts, among them J1 Power In, J2 RST, J3 RST, J4 RST, J5 RST, J6 Power In, SW1 RESET, SW2 PLAYER0, SW3 PLAYER1, SW4 MODE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

Commit message: PCB Fabrication Outputs
Parts:
- removed R17, R18, R3, R4, R5, R6, R7, R8: 510, Resistor_SMD:R_0805_2012Metric_Pad1.20x1.40mm_HandSolder, symbol Device:R_Small
- removed R20, R21: 4.7k, Resistor_SMD:R_0805_2012Metric_Pad1.20x1.40mm_HandSolder, symbol Device:R_Small
Connections:
- net MISO: now also SPI1.2 (Pin_2)
- net MOSI: now also SPI1.5 (Pin_5)
- net RXD: now also USART1.2 (Pin_2)
- net SCK: now also SPI1.4 (Pin_4)
- net SCL: now also I2C1.4 (Pin_4)
- net SDA: now also I2C1.2 (Pin_2)
- net TXD: now also USART1.5 (Pin_5)
- net V3V_0: now also RV1.3
- net V3V_1: now also RV2.3
- net XCK: now also USART1.4 (Pin_4)
Other:
- moved on the sheet: RV1
